Commit message: Plan for middle of gripper

File: src/description/urdf/panda_gaz.urdf (robot description, URDF)
Before this commit: robot panda, 12 links, 11 joints
Links:
- added link panda_leftfinger, mass 0.1; collision mesh filename=package://description/meshes/collision/finger.obj; visual mesh filename=package://description/meshes/visual/finger.obj
- added link panda_rightfinger, mass 0.1; collision mesh filename=package://description/meshes/collision/finger.obj; visual mesh filename=package://description/meshes/visual/finger.obj
Joints:
- added joint panda_finger_joint1: type fixed, parent panda_hand, child panda_leftfinger, origin xyz=0 0.04 0.0584 rpy=0 0 0, axis 0 1 0
- added joint panda_finger_joint2: type fixed, parent panda_hand, child panda_rightfinger, origin xyz=0 -0.04 0.0584 rpy=0 0 0, axis 0 -1 0
