Commit message: dual arm fingers + attach box p1/p2

File: src/description/urdf/TEST_gaz.urdf (robot description, URDF)
Before this commit: robot panda, 23 links, 22 joints
Links:
- added link panda1_leftfinger, mass 0.1; collision mesh filename=package://description/meshes/collision/finger.obj; visual mesh filename=package://description/meshes/visual/finger.obj
- added link panda1_rightfinger, mass 0.1; collision mesh filename=package://description/meshes/collision/finger.obj; visual mesh filename=package://description/meshes/visual/finger.obj
- added link panda2_leftfinger, mass 0.1; collision mesh filename=package://description/meshes/collision/finger.obj; visual mesh filename=package://description/meshes/visual/finger.obj
- added link panda2_rightfinger, mass 0.1; collision mesh filename=package://description/meshes/collision/finger.obj; visual mesh filename=package://description/meshes/visual/finger.obj
Joints:
- added joint panda1_finger_joint1: type fixed, parent panda1_hand, child panda1_leftfinger, origin xyz=0 0.04 0.0584 rpy=0 0 0, axis 0 1 0
- added joint panda1_finger_joint2: type fixed, parent panda1_hand, child panda1_rightfinger, origin xyz=0 -0.04 0.0584 rpy=0 0 0, axis 0 -1 0
- added joint panda2_finger_joint1: type fixed, parent panda2_hand, child panda2_leftfinger, origin xyz=0 0.04 0.0584 rpy=0 0 0, axis 0 1 0
- added joint panda2_finger_joint2: type fixed, parent panda2_hand, child panda2_rightfinger, origin xyz=0 -0.04 0.0584 rpy=0 0 0, axis 0 -1 0
