Commit message: reorga cleaner

File: src/bringup/urdf/panda1_gaz.urdf (robot description, URDF)
Before this commit: robot panda1, 12 links, 11 joints
Links:
- added link panda1_leftfinger, mass 0.1; collision mesh filename=package://bringup/meshes/collision/finger.obj; visual mesh filename=package://bringup/meshes/visual/finger.obj
- added link panda1_rightfinger, mass 0.1; collision mesh filename=package://bringup/meshes/collision/finger.obj; visual mesh filename=package://bringup/meshes/visual/finger.obj
- link panda1_hand: geometry collision mesh filename=package://bringup/meshes/collision/hand.obj; visual mesh filename=package://bringup/meshes/visual/hand.obj
- link panda1_link0: geometry collision mesh filename=package://bringup/meshes/collision/link0.obj; visual mesh filename=package://bringup/meshes/collision/link0.obj
- link panda1_link1: geometry collision mesh filename=package://bringup/meshes/collision/link1.obj; visual mesh filename=package://bringup/meshes/visual/link1.obj
- link panda1_link2: geometry collision mesh filename=package://bringup/meshes/collision/link2.obj; visual mesh filename=package://bringup/meshes/visual/link2.obj
- link panda1_link3: geometry collision mesh filename=package://bringup/meshes/collision/link3.obj; visual mesh filename=package://bringup/meshes/visual/link3.obj
- link panda1_link4: geometry collision mesh filename=package://bringup/meshes/collision/link4.obj; visual mesh filename=package://bringup/meshes/visual/link4.obj
- link panda1_link5: geometry collision mesh filename=package://bringup/meshes/collision/link5.obj; visual mesh filename=package://bringup/meshes/visual/link5.obj
- link panda1_link6: geometry collision mesh filename=package://bringup/meshes/collision/link6.obj; visual mesh filename=package://bringup/meshes/visual/link6.obj
- link panda1_link7: geometry collision mesh filename=package://bringup/meshes/collision/link7.obj; visual mesh filename=package://bringup/meshes/collision/link7.obj
Joints:
- added joint panda1_finger_joint1: type fixed, parent panda1_hand, child panda1_leftfinger, origin xyz=0 0.04 0.0584 rpy=0 0 0, axis 0 1 0
- added joint panda1_finger_joint2: type fixed, parent panda1_hand, child panda1_rightfinger, origin xyz=0 -0.04 0.0584 rpy=0 0 0, axis 0 -1 0

File: src/bringup/urdf/panda2_gaz.urdf (robot description, URDF)
Before this commit: robot panda2, 12 links, 11 joints
Links:
- added link panda2_leftfinger, mass 0.1; collision mesh filename=package://bringup/meshes/collision/finger.obj; visual mesh filename=package://bringup/meshes/visual/finger.obj
- added link panda2_rightfinger, mass 0.1; collision mesh filename=package://bringup/meshes/collision/finger.obj; visual mesh filename=package://bringup/meshes/visual/finger.obj
- link panda2_hand: geometry collision mesh filename=package://bringup/meshes/collision/hand.obj; visual mesh filename=package://bringup/meshes/visual/hand.obj
- link panda2_link0: geometry collision mesh filename=package://bringup/meshes/collision/link0.obj; visual mesh filename=package://bringup/meshes/collision/link0.obj
- link panda2_link1: geometry collision mesh filename=package://bringup/meshes/collision/link1.obj; visual mesh filename=package://bringup/meshes/visual/link1.obj
- link panda2_link2: geometry collision mesh filename=package://bringup/meshes/collision/link2.obj; visual mesh filename=package://bringup/meshes/visual/link2.obj
- link panda2_link3: geometry collision mesh filename=package://bringup/meshes/collision/link3.obj; visual mesh filename=package://bringup/meshes/visual/link3.obj
- link panda2_link4: geometry collision mesh filename=package://bringup/meshes/collision/link4.obj; visual mesh filename=package://bringup/meshes/visual/link4.obj
- link panda2_link5: geometry collision mesh filename=package://bringup/meshes/collision/link5.obj; visual mesh filename=package://bringup/meshes/visual/link5.obj
- link panda2_link6: geometry collision mesh filename=package://bringup/meshes/collision/link6.obj; visual mesh filename=package://bringup/meshes/visual/link6.obj
- link panda2_link7: geometry collision mesh filename=package://bringup/meshes/collision/link7.obj; visual mesh filename=package://bringup/meshes/collision/link7.obj
Joints:
- added joint panda2_finger_joint1: type fixed, parent panda2_hand, child panda2_leftfinger, origin xyz=0 0.04 0.0584 rpy=0 0 0, axis 0 1 0
- added joint panda2_finger_joint2: type fixed, parent panda2_hand, child panda2_rightfinger, origin xyz=0 -0.04 0.0584 rpy=0 0 0, axis 0 -1 0
