Commit message: obj drop orientation + human visual

File: src/bringup/urdf/panda2_robot_gaz.urdf (robot description, URDF)
Before this commit: robot panda2, 14 links, 13 joints
Links:
- link panda2_hand: geometry visual mesh filename=package://bringup/meshes/visual/hand.obj
- link panda2_leftfinger: geometry visual mesh filename=package://bringup/meshes/visual/finger.obj
- link panda2_link0: geometry visual mesh filename=package://bringup/meshes/collision/link0.obj
- link panda2_link1: geometry visual mesh filename=package://bringup/meshes/visual/link1.obj
- link panda2_link2: geometry visual mesh filename=package://bringup/meshes/visual/link2.obj
- link panda2_link3: geometry visual mesh filename=package://bringup/meshes/visual/link3.obj
- link panda2_link4: geometry visual mesh filename=package://bringup/meshes/visual/link4.obj
- link panda2_link5: geometry visual mesh filename=package://bringup/meshes/visual/link5.obj
- link panda2_link6: geometry visual mesh filename=package://bringup/meshes/visual/link6.obj
- link panda2_link7: geometry visual mesh filename=package://bringup/meshes/collision/link7.obj
- link panda2_rightfinger: geometry visual mesh filename=package://bringup/meshes/visual/finger.obj
