Commit message: remove collision (gaz:all moveit:hand)

File: src/bringup/urdf/panda1.urdf (robot description, URDF)
Before this commit: robot panda1, 12 links, 11 joints
Links:
- link panda1_hand: geometry visual mesh filename=package://bringup/meshes/visual/hand.obj

File: src/bringup/urdf/panda1_gaz.urdf (robot description, URDF)
Before this commit: robot panda1, 14 links, 13 joints
Links:
- link panda1_hand: geometry visual mesh filename=package://bringup/meshes/visual/hand.obj
- link panda1_leftfinger: geometry visual mesh filename=package://bringup/meshes/visual/finger.obj
- link panda1_link0: geometry visual mesh filename=package://bringup/meshes/collision/link0.obj
- link panda1_link1: geometry visual mesh filename=package://bringup/meshes/visual/link1.obj
- link panda1_link2: geometry visual mesh filename=package://bringup/meshes/visual/link2.obj
- link panda1_link3: geometry visual mesh filename=package://bringup/meshes/visual/link3.obj
- link panda1_link4: geometry visual mesh filename=package://bringup/meshes/visual/link4.obj
- link panda1_link5: geometry visual mesh filename=package://bringup/meshes/visual/link5.obj
- link panda1_link6: geometry visual mesh filename=package://bringup/meshes/visual/link6.obj
- link panda1_link7: geometry visual mesh filename=package://bringup/meshes/collision/link7.obj
- link panda1_rightfinger: geometry visual mesh filename=package://bringup/meshes/visual/finger.obj

File: src/bringup/urdf/panda2.urdf (robot description, URDF)
Before this commit: robot panda2, 12 links, 11 joints
Links:
- link panda2_hand: geometry visual mesh filename=package://bringup/meshes/visual/hand.obj

File: src/bringup/urdf/panda2_gaz.urdf (robot description, URDF)
Before this commit: robot panda2, 14 links, 13 joints
Links:
- link panda2_hand: geometry visual mesh filename=package://bringup/meshes/visual/hand.obj
- link panda2_leftfinger: geometry visual mesh filename=package://bringup/meshes/visual/finger.obj
- link panda2_link0: geometry visual mesh filename=package://bringup/meshes/collision/link0.obj
- link panda2_link1: geometry visual mesh filename=package://bringup/meshes/visual/link1.obj
- link panda2_link2: geometry visual mesh filename=package://bringup/meshes/visual/link2.obj
- link panda2_link3: geometry visual mesh filename=package://bringup/meshes/visual/link3.obj
- link panda2_link4: geometry visual mesh filename=package://bringup/meshes/visual/link4.obj
- link panda2_link5: geometry visual mesh filename=package://bringup/meshes/visual/link5.obj
- link panda2_link6: geometry visual mesh filename=package://bringup/meshes/visual/link6.obj
- link panda2_link7: geometry visual mesh filename=package://bringup/meshes/collision/link7.obj
- link panda2_rightfinger: geometry visual mesh filename=package://bringup/meshes/visual/finger.obj

Commit message: TEST new robot pose+hand+launch+reset

File: src/bringup/urdf/panda1.urdf (robot description, URDF)
Before this commit: robot panda1, 12 links, 11 joints
Joints:
- joint panda1_joint_world: origin xyz=0 0 0 rpy=0 0 0 -> xyz=0.2 0 0.3 rpy=0 0 0

File: src/bringup/urdf/panda2.urdf (robot description, URDF)
Before this commit: robot panda2, 12 links, 11 joints
Joints:
- joint panda2_joint_world: origin xyz=1.5 0 0 rpy=0 0 3.14159265 -> xyz=1.3 0 0.22 rpy=0 0 3.14159265

File: src/bringup/urdf/panda2_gaz.urdf (robot description, URDF)
Before this commit: robot panda2, 14 links, 13 joints
Links:
- link panda2_grasptarget: geometry visual mesh filename=package://bringup/meshes/human/hand.stl
- link panda2_hand: geometry 
