Commit message: place au services

File: src/bringup/urdf/panda2.urdf (robot description, URDF)
Before this commit: robot panda2, 12 links, 11 joints
Joints:
- joint panda2_joint_world: origin xyz=0 0 0 rpy=0 0 0 -> xyz=1.5 0 0 rpy=0 0 3.14159265

Commit message: initial poses

File: src/bringup/urdf/panda2.urdf (robot description, URDF)
Before this commit: robot panda2, 12 links, 11 joints
Joints:
- joint panda2_joint_world: origin xyz=1.3 0 0.22 rpy=0 0 3.14159265 -> xyz=1.3 0 0.3 rpy=0 0 3.14159265
