Commit message: launch files + worlds + move_hand

File: src/bringup/urdf/human_hand.urdf (robot description, URDF)
Before this commit: robot human_hand, 2 links, 1 joints
Joints:
- joint human_joint_world: origin xyz=1.3 0 0.3 rpy=0 0 3.14159265 -> xyz=0.0 0 0.0 rpy=0 0 0

Commit message: huge update

File: src/bringup/urdf/human_hand.urdf (robot description, URDF)
Before this commit: robot human_hand, 2 links, 1 joints
Links:
- link human_hand: geometry collision mesh filename=package://bringup/meshes/visual/hand.obj; visual mesh filename=package://bringup/meshes/human/hand.dae
Joints:
- joint human_joint_world: origin xyz=0.0 0 0.0 rpy=0 0 0 -> xyz=2 0.5 0.7 rpy=0 -0 3.14159

File: src/bringup/urdf/panda1.urdf (robot description, URDF)
Before this commit: robot panda1, 12 links, 11 joints
Joints:
- joint panda1_joint_world: origin xyz=0.2 0 0.3 rpy=0 0 0 -> xyz=0.2 0 0.6 rpy=0 0 0

Commit message: matching init hand pose in urdf w/ .world

File: src/bringup/urdf/human_hand.urdf (robot description, URDF)
Before this commit: robot human_hand, 2 links, 1 joints
Joints:
- joint human_joint_world: origin xyz=2 0.5 0.7 rpy=0 -0 3.14159 -> xyz=1.38 0.5 0.87 rpy=0 -0 3.14159
