Commit message: tiago

File: src/tiago/pal_gripper/pal_gripper_description/urdf/gripper.urdf.xacro (robot description, xacro)
@@ -150,5 +150,6 @@
                        soft_upper_limit="${0.045 - gripper_eps}" />
   </joint>
-  <xacro:pal_robotiq_grasping_frames prefix="${name}_" xyz="0 0 0.12"/>
+  <!-- <xacro:pal_robotiq_grasping_frames prefix="${name}_" xyz="0 0 0.12"/> -->
+  <xacro:pal_robotiq_grasping_frames prefix="${name}_" xyz="0 0 0.18"/>
   <xacro:gripper_simple_transmission name="${name}_left_finger" reduction="1.0"/>
   <xacro:gripper_simple_transmission name="${name}_right_finger" reduction="1.0"/>

File: src/tiago/pmb2_robot/pmb2_description/urdf/base/base.urdf.xacro (robot description, xacro)
@@ -38,8 +38,12 @@
       <inertial>
         <origin xyz="-0.00000106 0.00000109 0.0000387" rpy="0 0 0"/>
-        <mass value="28.26649"/>
+        <!-- <mass value="28.26649"/>
         <inertia ixx="0.465408937" ixy="0.002160024" ixz="-0.001760255"
                  iyy="0.483193291" iyz="-0.000655952"
-                 izz="0.550939703"/>
+                 izz="0.550939703"/> -->
+        <mass value="2826.649"/>
+        <inertia ixx="46.5408937" ixy="0.2160024" ixz="-0.1760255"
+                 iyy="48.3193291" iyz="-0.0655952"
+                 izz="55.0939703"/>
       </inertial>
       <visual>
@@ -67,4 +71,10 @@
       <child link="${name}_link" />
       <parent link="${name}_footprint"/>
+    </joint>
+    <link name="world" />
+    <joint name="joint_world" type="fixed">
+      <origin xyz="0.0 0 0.0" rpy="0 0 0" />
+      <parent link="world" />
+      <child link="${name}_footprint" />
     </joint>
   <!-- gazebo parameters are given here for base_link thru base_footprint -->

File: src/tiago/tiago_robot/tiago_description/urdf/arm/arm.urdf.xacro (robot description, xacro)
@@ -19,5 +19,5 @@
   <!--Constant parameters-->
   <xacro:property name="arm_friction"       value="1.0" />
-  <xacro:property name="arm_damping"        value="1.0" />
+  <xacro:property name="arm_damping"        value="10.0" />
   <xacro:property name="arm_1_max_vel"      value="1.95" />
   <xacro:property name="arm_2_max_vel"      value="1.95" />

File: src/tiago/tiago_robot/tiago_description/urdf/head/head.urdf.xacro (robot description, xacro)
@@ -101,4 +101,46 @@
       </collision>
     </link>
+    <link name="eye_r_link">
+      <inertial>
+        <origin xyz="0 0 0" rpy="0.00000 0.00000 0.00000"/>
+        <mass value="0.0"/>
+        <inertia ixx="0.00001" ixy="0.00001" ixz="0.00001"
+                 iyy="0.00001" iyz="0.00001"
+                 izz="0.00001"/>
+      </inertial>
+      <visual>
+        <origin xyz="0 0 0" rpy="0 0 0" />
+        <geometry>
+          <mesh filename="/home/afavier/blender/eye_r.dae" scale="1 1 1"/>
+        </geometry>
+        <material name="Black" />
+      </visual>
+    </link>
+    <joint name="$eye_r_joint" type="fixed">
+      <parent link="${name}_link"/>
+      <child link="eye_r_link"/>
+      <origin xyz="0.0 0.0 0.0"  rpy="0 0 0" />
+    </joint>
+    <link name="eye_l_link">
+      <inertial>
+        <origin xyz="0 0 0" rpy="0.00000 0.00000 0.00000"/>
+        <mass value="0.0"/>
+        <inertia ixx="0.00001" ixy="0.00001" ixz="0.00001"
+                 iyy="0.00001" iyz="0.00001"
+                 izz="0.00001"/>
+      </inertial>
+      <visual>
+        <origin xyz="0 0 0" rpy="0 0 0" />
+        <geometry>
+          <mesh filename="/home/afavier/blender/eye_l.dae" scale="1 1 1"/>
+        </geometry>
+        <material name="Black" />
+      </visual>
+    </link>
+    <joint name="$eye_l_joint" type="fixed">
+      <parent link="${name}_link"/>
+      <child link="eye_l_link"/>
+      <origin xyz="0.0 0.0 0.0"  rpy="0 0 0" />
+    </joint>
     <joint name="${name}_joint" type="revolute">
       <parent link="${parent}"/>

Commit message: fixed torso

File: src/tiago/pal_gripper/pal_gripper_description/urdf/gripper.urdf.xacro (robot description, xacro)
@@ -112,4 +112,9 @@
                        soft_upper_limit="${0.045 - gripper_eps}" />
   </joint>
+  <!-- <joint name="${name}_right_finger_joint" type="fixed">
+    <origin rpy="0 0 0" xyz="0. 0 0" />
+    <parent link="${name}_link" />
+    <child link="${name}_right_finger_link" />
+  </joint> -->
   <link name="${name}_left_finger_link">
     <inertial>
@@ -150,4 +155,9 @@
                        soft_upper_limit="${0.045 - gripper_eps}" />
   </joint>
+  <!-- <joint name="${name}_left_finger_joint" type="fixed">
+    <origin rpy="0 0 0" xyz="0. 0 0" />
+    <parent link="${name}_link" />
+    <child link="${name}_left_finger_link" />
+  </joint> -->
   <!-- <xacro:pal_robotiq_grasping_frames prefix="${name}_" xyz="0 0 0.12"/> -->
   <xacro:pal_robotiq_grasping_frames prefix="${name}_" xyz="0 0 0.18"/>

File: src/tiago/tiago_robot/tiago_description/robots/tiago.urdf.xacro (robot description, xacro)
@@ -27,5 +27,5 @@
     <xacro:arg name="no_safety_eps" default="false"/>
     <xacro:arg name="base_type" default="pmb2"/> <!-- pmb2, omni_base -->
-    <xacro:arg name="fixed_torso" default="false" />
+    <xacro:arg name="fixed_torso" default="true" />
     <xacro:property name="wrist_model" value="$(arg wrist_model)" />
     <xacro:property name="end_effector" value="$(arg end_effector)" />

File: src/tiago/tiago_robot/tiago_description/urdf/torso/torso.urdf.xacro (robot description, xacro)
@@ -129,5 +129,6 @@
     <joint name="${name}_lift_joint" type="fixed">
       <!-- Torso fixed height is set to half it's range -->
-      <origin rpy="0.0 0.0 0.0" xyz="0.0 0.0 0.772" />
+      <origin rpy="0.0 0.0 0.0" xyz="0.0 0.0 0.80" />
+      <!-- <origin rpy="0.0 0.0 0.0" xyz="0.0 0.0 0.30" /> -->
       <parent link="${name}_fixed_link" />
       <child link="${name}_lift_link" />

Commit message: remove gripper collision

File: src/tiago/pal_gripper/pal_gripper_description/urdf/gripper.urdf.xacro (robot description, xacro)
@@ -89,10 +89,10 @@
       <material name="Black"/>
     </visual>
-    <collision>
+    <!-- <collision>
       <origin rpy="0 0 3.1415" xyz="0.005 0 -0.165" />
       <geometry>
         <box size="0.01 0.05 0.11"/>
       </geometry>
-    </collision>
+    </collision> -->
   </link>
   <gazebo reference="${name}_right_finger_link">
@@ -132,10 +132,10 @@
       <material name="Black"/>
     </visual>
-    <collision>
+    <!-- <collision>
       <origin rpy="0 0 3.1415" xyz="-0.005 0 -0.165" />
       <geometry>
         <box size="0.01 0.05 0.11"/>
       </geometry>
-    </collision>
+    </collision> -->
   </link>
   <gazebo reference="${name}_left_finger_link">
