Commit message: tiago_eyes

File: src/tiago/tiago_robot/tiago_description/urdf/head/head.urdf.xacro (robot description, xacro)
@@ -101,5 +101,5 @@
       </collision>
     </link>
-    <link name="eye_r_link">
+    <link name="eyes_link">
       <inertial>
         <origin xyz="0 0 0" rpy="0.00000 0.00000 0.00000"/>
@@ -112,33 +112,12 @@
         <origin xyz="0 0 0" rpy="0 0 0" />
         <geometry>
-          <mesh filename="/home/afavier/blender/eye_r.dae" scale="1 1 1"/>
+          <mesh filename="/home/afavier/blender/tiago_eyes.dae" scale="1 1 1"/>
         </geometry>
         <material name="Black" />
       </visual>
     </link>
-    <joint name="$eye_r_joint" type="fixed">
+    <joint name="$eyes_joint" type="fixed">
       <parent link="${name}_link"/>
-      <child link="eye_r_link"/>
-      <origin xyz="0.0 0.0 0.0"  rpy="0 0 0" />
-    </joint>
-    <link name="eye_l_link">
-      <inertial>
-        <origin xyz="0 0 0" rpy="0.00000 0.00000 0.00000"/>
-        <mass value="0.0"/>
-        <inertia ixx="0.00001" ixy="0.00001" ixz="0.00001"
-                 iyy="0.00001" iyz="0.00001"
-                 izz="0.00001"/>
-      </inertial>
-      <visual>
-        <origin xyz="0 0 0" rpy="0 0 0" />
-        <geometry>
-          <mesh filename="/home/afavier/blender/eye_l.dae" scale="1 1 1"/>
-        </geometry>
-        <material name="Black" />
-      </visual>
-    </link>
-    <joint name="$eye_l_joint" type="fixed">
-      <parent link="${name}_link"/>
-      <child link="eye_l_link"/>
+      <child link="eyes_link"/>
       <origin xyz="0.0 0.0 0.0"  rpy="0 0 0" />
     </joint>

Commit message: blender meshes

File: src/tiago/tiago_robot/tiago_description/urdf/head/head.urdf.xacro (robot description, xacro)
@@ -112,5 +112,5 @@
         <origin xyz="0 0 0" rpy="0 0 0" />
         <geometry>
-          <mesh filename="/home/afavier/blender/tiago_eyes.dae" scale="1 1 1"/>
+          <mesh filename="/home/afavier/new_exec_sim_ws/src/simulator/meshes/tiago_eyes.dae" scale="1 1 1"/>
         </geometry>
         <material name="Black" />

Commit message: modifs file paths

File: src/tiago/tiago_robot/tiago_description/urdf/head/head.urdf.xacro (robot description, xacro)
@@ -112,5 +112,5 @@
         <origin xyz="0 0 0" rpy="0 0 0" />
         <geometry>
-          <mesh filename="/home/afavier/new_exec_sim_ws/src/simulator/meshes/tiago_eyes.dae" scale="1 1 1"/>
+          <mesh filename="/home/sshekhar/exec_simulator/src/simulator/meshes/tiago_eyes.dae" scale="1 1 1"/>
         </geometry>
         <material name="Black" />

Commit message: absolute path tag to replace

File: src/tiago/tiago_robot/tiago_description/urdf/head/head.urdf.xacro (robot description, xacro)
@@ -112,5 +112,5 @@
         <origin xyz="0 0 0" rpy="0 0 0" />
         <geometry>
-          <mesh filename="/home/afavier/new_exec_sim_ws/src/simulator/meshes/tiago_eyes.dae" scale="1 1 1"/>
+          <mesh filename="<absolute_path_to_replace>/src/simulator/meshes/tiago_eyes.dae" scale="1 1 1"/>
         </geometry>
         <material name="Black" />
